File: TransducerDriver/TransducerDriver.kicad_pcb (KiCad board)
At the start: 2 copper layers, 6 parts, among them Q1 IRF540N, Q2 IRF540N, T1 Transformer_SP_1S 1:10

Commit message: studies on transducer
Parts:
- removed Q1, Q2: IRF540N, Package_TO_SOT_THT:TO-220-3_Vertical
- removed Rshut1, Rshut2: 100, Resistors_THT:R_Axial_DIN0207_L6.3mm_D2.5mm_P10.16mm_Horizontal
- removed Rtrans1: 10K, Resistors_THT:R_Axial_DIN0207_L6.3mm_D2.5mm_P10.16mm_Horizontal
- removed T1: Transformer_SP_1S 1:10, Transformer_THT:Transformer_Toroid_Tapped_Horizontal_D10.5mm_Amidon-T37
- added C1: 159nF, Capacitors_THT:CP_Radial_D8.0mm_P5.00mm, F.Cu at (142.2, 48.3)
- added C2: 10nF, Capacitors_THT:C_Disc_D8.0mm_W5.0mm_P7.50mm, F.Cu at (144.8, 69.8)
- added C3: 0.1u, Capacitors_THT:C_Disc_D5.0mm_W2.5mm_P5.00mm, F.Cu at (58.4, 64.8)
- added C4: 0.1u, Capacitors_THT:C_Disc_D5.0mm_W2.5mm_P5.00mm, F.Cu at (95.2, 77.5)
- added D1: 1N4148, Diodes_THT:D_5W_P12.70mm_Horizontal, F.Cu at (129.5, 61.0)
- added D2: 1N4007, Diodes_THT:D_DO-35_SOD27_P10.16mm_Horizontal, F.Cu at (180.3, 101.6)
- added J1: ModSigJack, Pin_Headers:Pin_Header_Straight_1x02_Pitch2.54mm, F.Cu at (200.7, 110.5)
- added J2: BattJack, Pin_Headers:Pin_Header_Straight_1x01_Pitch2.54mm, F.Cu at (190.5, 118.1)
- added J3: BattJack, Pin_Headers:Pin_Header_Straight_1x01_Pitch2.54mm, F.Cu at (191.8, 91.4)
- added Q3: IRF540N, TO_SOT_Packages_THT:TO-220-3_Vertical, F.Cu at (182.9, 86.4)
- added Q4: IRF540N, TO_SOT_Packages_THT:TO-220-3_Vertical, F.Cu at (201.9, 86.4)
- added R1: 101, Resistors_THT:R_Axial_DIN0309_L9.0mm_D3.2mm_P12.70mm_Horizontal, F.Cu at (82.5, 54.6)
- added R10: 2Khom, Resistors_THT:R_Axial_DIN0309_L9.0mm_D3.2mm_P12.70mm_Horizontal, F.Cu at (108.0, 106.7)
- added R11: 1Kohm, Resistors_THT:R_Axial_DIN0309_L9.0mm_D3.2mm_P12.70mm_Horizontal, F.Cu at (128.3, 106.7)
- added R6: 4K, Resistors_THT:R_Axial_DIN0309_L9.0mm_D3.2mm_P12.70mm_Horizontal, F.Cu at (121.9, 22.9)
- added R7: 4K, Resistors_THT:R_Axial_DIN0309_L9.0mm_D3.2mm_P12.70mm_Horizontal, F.Cu at (106.7, 22.9)
- added R8: 101, Resistors_THT:R_Axial_DIN0309_L9.0mm_D3.2mm_P12.70mm_Horizontal, F.Cu at (109.2, 54.6)
- added R9: 530, Resistors_THT:R_Axial_DIN0309_L9.0mm_D3.2mm_P12.70mm_Horizontal, F.Cu at (72.4, 108.0)
- added Rshut3: 0.01, Resistors_THT:R_Axial_DIN0207_L6.3mm_D2.5mm_P10.16mm_Horizontal, F.Cu at (191.8, 71.1)
- added T2: Transformer_SP_1S 1:10, Transformers_THT:Transformer_Toroid_Tapped_Horizontal_D14.0mm_Amidon-T50, F.Cu at (184.2, 62.2)
- added U1: INA217, Housings_DIP:DIP-8_W7.62mm, F.Cu at (90.2, 52.1)
- added U2: INA217, Housings_DIP:DIP-8_W7.62mm, F.Cu at (116.8, 52.1)
- added U3: TC427, Housings_DIP:DIP-8_W7.62mm_LongPads, F.Cu at (186.7, 105.4)
- added Y1: Crystal, Wire_Connections_Bridges:WireConnection_2.50mmDrill, F.Cu at (87.6, 67.3)
- added Y2: Crystal, Wire_Connections_Bridges:WireConnection_2.50mmDrill, F.Cu at (194.3, 30.5)
Routing:
- net /Vref: track 0.00 -> 60.2 mm
- net Net-(U1-Pad6): track 0.00 -> 28.8 mm
- net Net-(C1-Pad2): track 0.00 -> 18.2 mm
- net Net-(Q1-Pad2): track 14.0 -> 0.00 mm
- net Net-(Rshut2-Pad1): track 10.3 -> 0.00 mm
- net Net-(Rshut1-Pad1): track 10.2 -> 0.00 mm
- net Net-(Q2-Pad2): track 10.2 -> 0.00 mm
- net (no net): track 9.73 -> 0.00 mm
- net Net-(R1-Pad1): track 0.00 -> 9.29 mm
- net Net-(R8-Pad1): track 0.00 -> 9.29 mm
- net Net-(R8-Pad2): track 0.00 -> 8.67 mm
- net Net-(R1-Pad2): track 0.00 -> 8.67 mm
- net GND: track 8.17 -> 0.00 mm
- added copper zone on B.Cu, net GND
