File: TransducerDriver/_saved_TransducerDriver.sch (KiCad schematic (older format))
At the start: 49 parts, among them J1 ModSigJack, J2 BattJack+, J3 BattJack-, Q3 IRF540N, Q4 IRF540N, T1 Transformer_SP_1S 1:10, U1 TL082, U2 INA217-Amplifier_Instrumentat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, U3 TC427, U4 LM4562, Y1 Crystal, Y2 Fish Finder

Commit message: more impedance data
Other:
- note added: "Z is imagenary part\n of impedance"
- moved on the sheet: C2In1, C2In2, C2out1, C3, C4, Cadc1, Cb1, Cb?, Cenv1, Cg1, Cgnd2, Cref2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
