File: TransducerDriver/_autosave-TransducerDriver.sch (KiCad schematic (older format))
At the start: 53 parts, among them J1 ModSigJack, J2 BattJack+, J3 BattJack-, Q3 IRF540N, Q4 IRF540N, T1 Transformer_SP_1S 1:10, T2 Transformer_SP_1S 1:10, T3 Transformer_SP_1S 1:10, U1 TL082, U2 INA217-Amplifier_Instrumentat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, U3 TC427, U4 LM4562, Y1 Crystal, Y2 Fish Finder, Y3 FishFinder, Y4 FishFinder

Commit message: more mod on circuits
Parts:
- Rb1: value 5K -> 500ohm
Connections:
- net ADCinput: no longer Dz1.1 (K)
Other:
- note removed: "6Kohm Internal \nR. Is it High \noutput Impedance?"
- moved on the sheet: Dz1
Changed lines of the file:
@@
 EESchema Schematic File Version 4
 LIBS:TransducerDriver-cache
-EELAYER 26 0
+EELAYER 30 0
 EELAYER END
 $Descr A4 11693 8268
@@
 Wire Notes Line
 	800  3750 1500 3750
-Text Notes 750  4250 0    50   ~ 0
+Text Notes 850  4200 0    50   ~ 0
 Fish Finder
 $Comp
@@
 P 2300 6050
 F 0 "Rb1" H 2370 6096 50  0000 L CNN
-F 1 "5K" H 2370 6005 50  0000 L CNN
+F 1 "500ohm" H 2370 6005 50  0000 L CNN
 F 2 "Resistors_THT:R_Axial_DIN0309_L9.0mm_D3.2mm_P12.70mm_Horizontal" V 2230 6050 50  0001 C CNN
 F 3 "~" H 2300 6050 50  0001 C CNN
@@
 	0    1    1    0
 $EndComp
-Text Notes 3800 4100 0    50   ~ 0
-6Kohm Internal \nR. Is it High \noutput Impedance?
 Text Notes 5350 5550 0    50   ~ 0
 10Khz HP filter\n0.1uF 1Kohm
@@
 Text Notes 4850 3550 0    67   Italic 13
 Two Options for second stage
-$Comp
-L Device:D_Zener Dz1
-U 1 1 5E645861
-P 10150 4250
-F 0 "Dz1" V 10150 4400 50  0000 C CNN
-F 1 "3.3V" V 10250 4400 50  0000 C CNN
-F 2 "" H 10150 4250 50  0001 C CNN
-F 3 "~" H 10150 4250 50  0001 C CNN
-	1    10150 4250
-	0    1    1    0
-$EndComp
-$Comp
-L power:GND #PWR014
-U 1 1 5E64625D
-P 10150 4400
-F 0 "#PWR014" H 10150 4150 50  0001 C CNN
-F 1 "GND" H 10155 4227 50  0000 C CNN
-F 2 "" H 10150 4400 50  0001 C CNN
-F 3 "" H 10150 4400 50  0001 C CNN
-	1    10150 4400
-	1    0    0    -1
-$EndComp
-Text GLabel 10250 3900 2    50   Input ~ 0
-ADCinput
-Wire Wire Line
-	10150 4100 10150 3800
 Text GLabel 8700 5500 0    50   Input ~ 0
 ADCinput
@@
 Text Notes 9700 3750 0    50   ~ 0
 Potential\nVariable \nGain
-Wire Wire Line
-	9550 3800 10150 3800
 Connection ~ 9550 3800
-Connection ~ 10150 3800
 Text Notes 7950 3700 0    67   Italic 13
 Envelope\nDetector
@@
 $EndComp
 Wire Wire Line
-	10150 3800 10200 3800
-Wire Wire Line
-	10250 3900 10200 3900
-Wire Wire Line
-	10200 3900 10200 3800
-Connection ~ 10200 3800
-Wire Wire Line
-	10200 3800 10350 3800
-Wire Wire Line
 	4450 1250 4450 2050
 $Comp
@@
 Wire Wire Line
 	9250 3800 9550 3800
+Wire Wire Line
+	10200 3800 10350 3800
+Connection ~ 10200 3800
+$Comp
+L Device:D_Zener Dz1
+U 1 1 5E645861
+P 11000 4750
+F 0 "Dz1" V 11000 4900 50  0000 C CNN
+F 1 "3.3V" V 11100 4900 50  0000 C CNN
+F 2 "" H 11000 4750 50  0001 C CNN
+F 3 "~" H 11000 4750 50  0001 C CNN
+	1    11000 4750
+	0    1    1    0
+$EndComp
+$Comp
+L power:GND #PWR014
+U 1 1 5E64625D
+P 11000 4900
+F 0 "#PWR014" H 11000 4650 50  0001 C CNN
+F 1 "GND" H 11005 4727 50  0000 C CNN
+F 2 "" H 11000 4900 50  0001 C CNN
+F 3 "" H 11000 4900 50  0001 C CNN
+	1    11000 4900
+	1    0    0    -1
+$EndComp
+Wire Wire Line
+	11000 4600 11000 4300
+Wire Wire Line
+	10200 3900 10200 3800
+Wire Wire Line
+	10250 3900 10200 3900
+Text GLabel 10250 3900 2    50   Input ~ 0
+ADCinput
+Wire Wire Line
+	9550 3800 10200 3800
 $EndSCHEMATC
