File: TransducerDriver/TransducerDriver.sch (KiCad schematic (older format))
At the start: 49 parts, among them J1 ModSigJack, J2 BattJack+, J3 BattJack-, Q3 IRF540N, Q4 IRF540N, T1 Transformer_SP_1S 1:10, U1 TL082, U2 INA217-Amplifier_Instrumentat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, U3 TC427, U4 LM4562, Y1 Crystal, Y2 Fish Finder

Commit message: impedance calculation done
Parts:
- added Rm3, Rm4: Zmatch, Resistors_THT:R_Axial_DIN0309_L9.0mm_D3.2mm_P12.70mm_Horizontal, symbol Device:R
- added T3: Transformer_SP_1S 1:10, Transformers_THT:Transformer_Toroid_Tapped_Horizontal_D14.0mm_Amidon-T50, symbol Device:Transformer_SP_1S
- added Y4: FishFinder, Wire_Connections_Bridges:WireConnection_2.50mmDrill, symbol Device:Crystal
- gave numbers to parts that had none: 3
- renumbered Dvref to Dvref1
Connections:
- net at T2.5 (S2): now also Rm4.2; no longer Y3.1
- new net: Rm4.1, Y3.1
- new net: Rm3.1, T3.4 (S1), Y4.2
- new net: Rm3.2, T3.5 (S2), Y4.1
Other:
- note added: "Z is imagenary part\n of impedance"
- note added: "Zmatch = (Zsource * Zfish) / (Zfish - Zsource)"
- moved on the sheet: C2In1, C2In2, C2out1, C3, C4, Cadc1, Cb1, Cb2, Cenv1, Cg1, Cgnd2, Cref2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

Commit message: more calculation
Connections:
- net Stage2Out: now also Rf2.1, U4.1
Other:
- note added: "0.8Khz HP filter\n0.1uF 2Kohm"
- note added: "Impedance Match"
- note added: "low Rin2 to force \na Vref DC bias"
- note removed: "Rin2 same as R2 \nlimit input bias current"
- note removed: "Z is imagenary part\n of impedance"
- moved on the sheet: Rm4, T2, Y3
Changed lines of the file:
@@
 Title "Acoustic Link Analog circuits"
 Date "2020-02-11"
-Rev "2.1"
+Rev "2.3"
 Comp ""
 Comment1 "Leo Chen"
@@
 Text Notes 6500 5050 0    50   ~ 0
 X cgnd1<<Rg2 \nF = 20Khz\nC = 0.47uF \nXc = 17ohm
-Text Notes 5050 3850 0    50   ~ 0
-Rin2 same as R2 \nlimit input bias current
+Text Notes 5450 3800 0    50   ~ 0
+low Rin2 to force \na Vref DC bias
 $Comp
 L TransducerDriver-rescue:INA217-Amplifier_Instrumentation U2
@@
 L Device:Transformer_SP_1S T2
 U 1 1 5E55647C
-P 8900 1100
-F 0 "T2" H 8900 650 50  0000 C CNN
-F 1 "Transformer_SP_1S 1:10" H 8900 800 50  0000 C CNN
-F 2 "Transformers_THT:Transformer_Toroid_Tapped_Horizontal_D14.0mm_Amidon-T50" H 8900 1100 50  0001 C CNN
-F 3 "~" H 8900 1100 50  0001 C CNN
-	1    8900 1100
+P 8900 1250
+F 0 "T2" H 8900 800 50  0000 C CNN
+F 1 "Transformer_SP_1S 1:10" H 8900 950 50  0000 C CNN
+F 2 "Transformers_THT:Transformer_Toroid_Tapped_Horizontal_D14.0mm_Amidon-T50" H 8900 1250 50  0001 C CNN
+F 3 "~" H 8900 1250 50  0001 C CNN
+	1    8900 1250
 	1    0    0    -1
 $EndComp
@@
 L Device:Crystal Y3
 U 1 1 5E556485
-P 10350 1150
-F 0 "Y3" V 10304 1281 50  0000 L CNN
-F 1 "FishFinder" V 10395 1281 50  0000 L CNN
-F 2 "Wire_Connections_Bridges:WireConnection_2.50mmDrill" H 10350 1150 50  0001 C CNN
-F 3 "~" H 10350 1150 50  0001 C CNN
-	1    10350 1150
+P 10350 1300
+F 0 "Y3" V 10304 1431 50  0000 L CNN
+F 1 "FishFinder" V 10395 1431 50  0000 L CNN
+F 2 "Wire_Connections_Bridges:WireConnection_2.50mmDrill" H 10350 1300 50  0001 C CNN
+F 3 "~" H 10350 1300 50  0001 C CNN
+	1    10350 1300
 	0    1    1    0
 $EndComp
@@
 	6350 450  6350 3250
 Wire Notes Line
-	9500 750  9600 750
-Wire Notes Line
-	9600 750  9600 1450
-Wire Notes Line
-	9600 1450 9500 1450
-Text Notes 9300 850  0    50   ~ 0
+	9500 900  9600 900
+Wire Notes Line
+	9600 900  9600 1600
+Wire Notes Line
+	9600 1600 9500 1600
+Text Notes 9300 1000 0    50   ~ 0
 Zsource
 Wire Notes Line
-	9850 750  9750 750
-Wire Notes Line
-	9750 750  9750 1450
-Wire Notes Line
-	9750 1450 9850 1450
-Text Notes 9800 850  0    50   ~ 0
+	9850 900  9750 900
+Wire Notes Line
+	9750 900  9750 1600
+Wire Notes Line
+	9750 1600 9850 1600
+Text Notes 9800 1000 0    50   ~ 0
 Zload=Zfish+Zmatch
 Wire Wire Line
-	10350 900  10350 1000
-Wire Wire Line
-	9300 1300 10350 1300
-Text Notes 9250 1600 0    50   ~ 0
+	10350 1050 10350 1150
+Wire Wire Line
+	9300 1450 10350 1450
+Text Notes 9250 1750 0    50   ~ 0
 Zmatch = Zsource - Zfish
 Text Notes 6900 3100 0    39   ~ 0
@@
 L Device:R Rm4
 U 1 1 5E59E5EC
-P 10050 900
-F 0 "Rm4" V 10050 850 50  0000 L CNN
-F 1 "Zmatch" V 10150 750 50  0000 L CNN
-F 2 "Resistors_THT:R_Axial_DIN0309_L9.0mm_D3.2mm_P12.70mm_Horizontal" V 9980 900 50  0001 C CNN
-F 3 "~" H 10050 900 50  0001 C CNN
-	1    10050 900
-	0    1    1    0
-$EndComp
-Wire Wire Line
-	10350 900  10200 900
-Wire Wire Line
-	9900 900  9300 900
+P 10050 1050
+F 0 "Rm4" V 10050 1000 50  0000 L CNN
+F 1 "Zmatch" V 10150 900 50  0000 L CNN
+F 2 "Resistors_THT:R_Axial_DIN0309_L9.0mm_D3.2mm_P12.70mm_Horizontal" V 9980 1050 50  0001 C CNN
+F 3 "~" H 10050 1050 50  0001 C CNN
+	1    10050 1050
+	0    1    1    0
+$EndComp
+Wire Wire Line
+	10350 1050 10200 1050
+Wire Wire Line
+	9900 1050 9300 1050
 Wire Notes Line
 	8150 450  8150 3250
@@
 Text Notes 8750 3000 0    50   ~ 0
 Zmatch = (Zsource * Zfish) / (Zfish - Zsource)
-Text Notes 8200 650  0    50   Italic 0
-Z is imagenary part\n  of impedance
 $Comp
 L Device:R Rm3
@@
 Wire Wire Line
 	9950 2600 10350 2600
+Text Notes 4950 4350 0    50   ~ 0
+0.8Khz HP filter\n0.1uF 2Kohm
+Text GLabel 6750 4150 2    50   Input ~ 0
+Stage2Out
+Text Notes 8200 700  0    157  ~ 31
+Impedance Match
 $EndSCHEMATC

Commit message: more mod on circuits
Parts:
- added Rdown: 10K, Resistors_THT:R_Axial_DIN0309_L9.0mm_D3.2mm_P12.70mm_Horizontal, symbol Device:R
- Cenv1: value 10nf -> 0.1uF
Connections:
- net GND: now also Rdown.2
- net Prob: now reaches C2out1.1, D1.1 (K)
- net Prob: now also Rdown.1
Other:
- note added: "1/80Khz = 12.5us\n1/1Khz = 1ms\npick 200us as time constant"
- note removed: "min Fcarr = 40Khz \nmax Fmod = 1Khz \n10nF 2Kohm\nFc = 8Kohm"
- moved on the sheet: Cadc1, Radc1
Changed lines of the file:
@@
 	2200 2200 1900 2200
-Wire Wire Line
-	3500 2000 3600 2000
 Wire Wire Line
 	3600 2000 3600 1800
@@
 Wire Wire Line
 	10150 4100 10150 3800
-Text GLabel 8700 5150 0    50   Input ~ 0
+Text GLabel 8700 5500 0    50   Input ~ 0
 ADCinput
 $Comp
 L Device:R Radc1
 U 1 1 5E653FDE
-P 8950 5150
-F 0 "Radc1" V 8850 5050 50  0000 L CNN
-F 1 "2.5K" V 9050 5050 50  0000 L CNN
-F 2 "Resistors_THT:R_Axial_DIN0309_L9.0mm_D3.2mm_P12.70mm_Horizontal" V 8880 5150 50  0001 C CNN
-F 3 "~" H 8950 5150 50  0001 C CNN
-	1    8950 5150
+P 8950 5500
+F 0 "Radc1" V 8850 5400 50  0000 L CNN
+F 1 "2.5K" V 9050 5400 50  0000 L CNN
+F 2 "Resistors_THT:R_Axial_DIN0309_L9.0mm_D3.2mm_P12.70mm_Horizontal" V 8880 5500 50  0001 C CNN
+F 3 "~" H 8950 5500 50  0001 C CNN
+	1    8950 5500
 	0    1    1    0
 $EndComp
@@
 L Device:C Cadc1
 U 1 1 5E654634
-P 9200 5400
-F 0 "Cadc1" H 9085 5354 50  0000 R CNN
-F 1 "10pf" H 9085 5445 50  0000 R CNN
-F 2 "Capacitors_THT:C_Disc_D8.0mm_W5.0mm_P7.50mm" H 9238 5250 50  0001 C CNN
-F 3 "~" H 9200 5400 50  0001 C CNN
-	1    9200 5400
+P 9200 5750
+F 0 "Cadc1" H 9085 5704 50  0000 R CNN
+F 1 "10pf" H 9085 5795 50  0000 R CNN
+F 2 "Capacitors_THT:C_Disc_D8.0mm_W5.0mm_P7.50mm" H 9238 5600 50  0001 C CNN
+F 3 "~" H 9200 5750 50  0001 C CNN
+	1    9200 5750
 	-1   0    0    1
 $EndComp
 Wire Wire Line
-	9100 5150 9200 5150
-Wire Wire Line
-	9200 5150 9200 5250
-Wire Wire Line
-	8800 5150 8700 5150
+	9100 5500 9200 5500
+Wire Wire Line
+	9200 5500 9200 5600
+Wire Wire Line
+	8800 5500 8700 5500
 $Comp
 L power:GND #PWR012
 U 1 1 5E65CE66
-P 9200 5550
-F 0 "#PWR012" H 9200 5300 50  0001 C CNN
-F 1 "GND" H 9205 5377 50  0000 C CNN
-F 2 "" H 9200 5550 50  0001 C CNN
-F 3 "" H 9200 5550 50  0001 C CNN
-	1    9200 5550
-	1    0    0    -1
-$EndComp
-Wire Notes Line
-	8750 4950 8750 5800
-Wire Notes Line
-	8750 5800 9700 5800
-Wire Notes Line
-	9700 5800 9700 4950
-Wire Notes Line
-	9700 4950 8750 4950
-Text Notes 9100 5100 0    59   Italic 12
+P 9200 5900
+F 0 "#PWR012" H 9200 5650 50  0001 C CNN
+F 1 "GND" H 9205 5727 50  0000 C CNN
+F 2 "" H 9200 5900 50  0001 C CNN
+F 3 "" H 9200 5900 50  0001 C CNN
+	1    9200 5900
+	1    0    0    -1
+$EndComp
+Wire Notes Line
+	8750 5300 8750 6150
+Wire Notes Line
+	8750 6150 9700 6150
+Wire Notes Line
+	9700 6150 9700 5300
+Wire Notes Line
+	9700 5300 8750 5300
+Text Notes 9100 5450 0    59   Italic 12
 ADC internal
-$Comp
-L Device:C_Small Cenv1
-U 1 1 5E672EB5
-P 9250 4100
-F 0 "Cenv1" H 9260 4170 50  0000 L CNN
-F 1 "10nf" H 9260 4020 50  0000 L CNN
-F 2 "Capacitors_THT:C_Disc_D5.0mm_W2.5mm_P5.00mm" H 9250 4100 50  0001 C CNN
-F 3 "~" H 9250 4100 50  0001 C CNN
-	1    9250 4100
-	-1   0    0    -1
-$EndComp
 Wire Wire Line
 	9250 3800 9250 4000
@@
 U 1 1 5E67C655
 P 8550 3800
-F 0 "C2out1" V 8750 3750 50  0000 L CNN
-F 1 "0.1u" V 8650 3750 50  0000 L CNN
+F 0 "C2out1" V 8750 3650 50  0000 L CNN
+F 1 "0.1u" V 8650 3700 50  0000 L CNN
 F 2 "Capacitors_THT:C_Disc_D5.0mm_W2.5mm_P5.00mm" H 8550 3800 50  0001 C CNN
 F 3 "~" H 8550 3800 50  0001 C CNN
@@
 	0    1    -1   0
 $EndComp
-Text Notes 8350 4550 0    50   ~ 0
-min Fcarr = 40Khz \nmax Fmod = 1Khz \n10nF 2Kohm\nFc = 8Kohm
 Wire Wire Line
 	8350 3800 8450 3800
 Wire Wire Line
-	8650 3800 8750 3800
+	8650 3800 8700 3800
 Wire Notes Line
 	9650 3850 10100 3850
 Wire Notes Line
-	10100 3850 10100 3500
-Wire Notes Line
-	10100 3500 9650 3500
-Wire Notes Line
-	9650 3850 9650 3500
+	10100 3850 10100 3450
+Wire Notes Line
+	10100 3450 9650 3450
+Wire Notes Line
+	9650 3850 9650 3450
 Text Notes 9700 3750 0    50   ~ 0
 Potential\nVariable \nGain
-Wire Wire Line
-	9250 3800 9550 3800
 Wire Wire Line
 	9550 3800 10150 3800
@@
 Envelope\nDetector
 Wire Notes Line
-	7850 3450 10650 3450
-Wire Notes Line
-	10650 3450 10650 4650
-Wire Notes Line
-	10650 4650 7850 4650
-Wire Notes Line
-	7850 4650 7850 3450
+	7850 3350 10650 3350
+Wire Notes Line
+	10650 3350 10650 4900
+Wire Notes Line
+	10650 4900 7850 4900
+Wire Notes Line
+	7850 4900 7850 3350
 $Comp
 L Connector:Conn_01x01_Male Jadc1
@@
 	3200 3700 3550 3700
 Wire Wire Line
-	5300 1850 5600 1850
-Wire Wire Line
 	5300 2250 5600 2250
 Text GLabel 2000 4400 0    50   Input ~ 0
@@
 Text Notes 8200 700  0    157  ~ 31
 Impedance Match
+Wire Wire Line
+	3500 2000 3600 2000
+Wire Wire Line
+	5300 1850 5600 1850
+$Comp
+L Device:C_Small Cenv1
+U 1 1 5E672EB5
+P 9250 4100
+F 0 "Cenv1" H 9260 4170 50  0000 L CNN
+F 1 "0.1uF" H 9260 4020 50  0000 L CNN
+F 2 "Capacitors_THT:C_Disc_D5.0mm_W2.5mm_P5.00mm" H 9250 4100 50  0001 C CNN
+F 3 "~" H 9250 4100 50  0001 C CNN
+	1    9250 4100
+	-1   0    0    -1
+$EndComp
+Text Notes 8000 4800 0    50   ~ 0
+1/80Khz = 12.5us\n1/1Khz = 1ms\npick 200us as time constant
+$Comp
+L Device:R Rdown
+U 1 1 5E5726AC
+P 8700 4150
+F 0 "Rdown" H 8770 4196 50  0000 L CNN
+F 1 "10K" H 8770 4105 50  0000 L CNN
+F 2 "Resistors_THT:R_Axial_DIN0309_L9.0mm_D3.2mm_P12.70mm_Horizontal" V 8630 4150 50  0001 C CNN
+F 3 "~" H 8700 4150 50  0001 C CNN
+	1    8700 4150
+	1    0    0    -1
+$EndComp
+$Comp
+L power:GND #PWR?
+U 1 1 5E57295E
+P 8700 4300
+F 0 "#PWR?" H 8700 4050 50  0001 C CNN
+F 1 "GND" H 8705 4127 50  0000 C CNN
+F 2 "" H 8700 4300 50  0001 C CNN
+F 3 "" H 8700 4300 50  0001 C CNN
+	1    8700 4300
+	1    0    0    -1
+$EndComp
+Wire Wire Line
+	8700 3800 8700 4000
+Connection ~ 8700 3800
+Wire Wire Line
+	8700 3800 8750 3800
+Text GLabel 8700 3500 1    50   Input ~ 0
+Prob
+Wire Wire Line
+	9250 3800 9550 3800
+Wire Wire Line
+	8700 3500 8700 3800
 $EndSCHEMATC

Commit message: more measurement and schmatic update
Parts:
- removed C2In1, Cref2: 0.1u, Capacitors_THT:C_Disc_D5.0mm_W2.5mm_P5.00mm, symbol Device:C_Small
- removed Cg1: 0.47uF, Capacitors_THT:C_Disc_D5.0mm_W2.5mm_P5.00mm, symbol Device:C_Small
- removed Rf2: 200K, Resistors_THT:R_Axial_DIN0309_L9.0mm_D3.2mm_P12.70mm_Horizontal, symbol Device:R
- removed Rg1, Rin2: 2K, Resistors_THT:R_Axial_DIN0309_L9.0mm_D3.2mm_P12.70mm_Horizontal, symbol Device:R
- removed unit 1 of U4
- added C2lp1: ?, Capacitors_THT:C_Disc_D5.0mm_W2.5mm_P5.00mm, symbol Device:C_Small
- added Cbp1: 0.1uF, symbol Device:C_Small
- added Cbp2: 10uF, symbol Device:C_Small
- added Dprot1, Dprot2: 1N4148, symbol Device:D_Small
- added Lbatt1: 300uH, symbol Device:L_Small
- added Lbatt?: 5.72uH, symbol Device:L_Small
- renumbered Rdown to Rdown1
Connections:
- net +BATT: now also Cbp1.1, Cbp2.1, Lbatt1.1; no longer T1.2 (PM)
- net GND: now also Cbp1.2, Cbp2.2
- net Stage2Out: now also C2lp1.1
- net at Q3.1 (G), U3.7 (OUT_A): now also Dprot2.2 (A)
- net at T1.5 (S2): now also Lbatt?.1; no longer Y2.1
- net at Q4.1 (G), U3.5 (OUT_B): now also Dprot1.2 (A)
- net at D2.1 (K), U3.6 (Vdd): now also Dprot1.1 (K), Dprot2.1 (K)
- net at R2F1.2, R2G1.1, U4.6 (-): now also C2lp1.2
- new net: Lbatt1.2, T1.2 (PM)
- new net: Lbatt?.2, Y2.1
Other:
- note added: "Inverting"
- note added: "Second stage"
- note removed: "0.8Khz HP filter\n0.1uF 2Kohm"
- note removed: "Inverting \nSimple Vref"
- note removed: "Non-Inverting\nHigh Impedance"
- note removed: "Two Options for second stage"
- note removed: "X cgnd1<<Rg2 \nF = 20Khz\nC = 0.47uF \nXc = 17ohm"
- note removed: "low Rin2 to force \na Vref DC bias"
- moved on the sheet: C2In2, Cgnd2, D2, Q3, Q4, R2F1, R2G1, T1, U4B, U4C, Y2

Commit message: final clean up
Parts:
- removed C2out1: 0.1u, Capacitors_THT:C_Disc_D5.0mm_W2.5mm_P5.00mm, symbol Device:C_Small
- removed D1: 1N4148, Diodes_THT:D_5W_P12.70mm_Horizontal, symbol pspice:DIODE
- removed Dz1: 3.3V, symbol Device:D_Zener
- removed Jadc1: connADC, symbol Connector:Conn_01x01_Male
- removed Lbatt1: 300uH, symbol Device:L_Small
- removed Rdown1: 10K, Resistors_THT:R_Axial_DIN0309_L9.0mm_D3.2mm_P12.70mm_Horizontal, symbol Device:R
- added C1, C2, C5: 470uF, symbol Device:CP
- added C2out2: 0.1u, Capacitors_THT:C_Disc_D5.0mm_W2.5mm_P5.00mm, symbol Device:C_Small
- added D3: 1N4148, Diodes_THT:D_5W_P12.70mm_Horizontal, symbol pspice:DIODE
- added Dz4: 3.3V, symbol Device:D_Zener
- added Jadc2: connADC, symbol Connector:Conn_01x01_Male
- added Rblock1: 0.1ohm, Resistors_THT:R_Axial_DIN0207_L6.3mm_D2.5mm_P10.16mm_Horizontal, symbol Device:R
- added Rd1: 1K, Resistors_THT:R_Axial_DIN0309_L9.0mm_D3.2mm_P12.70mm_Horizontal, symbol Device:R
- added Rlim2: 100, Resistors_THT:R_Axial_DIN0309_L9.0mm_D3.2mm_P12.70mm_Horizontal, symbol Device:R
- added unit 3 of U1
- added unit 1 of U4
- Cbp1: value 0.1uF -> 10uF
- Cenv1: value 0.1uF -> 1n
- Renv1: value 2K -> 300K
- gave numbers to parts that had none: 1
Connections:
- net +BATT: now also C2.1, C5.1, Rblock1.1, U1.8 (V+); no longer Cbp1.1
- net ADCinput: now also Dz4.1 (K), Jadc2.1 (Pin_1), Rlim2.1; no longer Cenv1.1, Renv1.1
- net GND: now also C1.2, C2.2, C5.2, Dz4.2 (A), Rd1.2, U1.4 (V-)
- net Stage2Out: now also C2out2.2
- net at T1.2 (PM): now also Rblock1.2
- net at D2.1 (K), Dprot1.1 (K), Dprot2.1 (K)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: now also Cbp1.1, C1.1
- new net: C2out2.1, D3.1 (K), Rd1.1
- new net: Cenv1.1, D3.2 (A), Renv1.1, U4.3 (+)
- new net: Rlim2.2, U4.1, U4.2 (-)
Other:
- note added: "First Stage Diff Amp"
- note added: "Second stage Inverting Amp"
- note removed: "1/80Khz = 12.5us\n1/1Khz = 1ms\npick 200us as time constant"
- note removed: "First Stage \nDiff Amp"
- note removed: "Inverting"
- note removed: "Potential\nVariable \nGain"
- note removed: "Second stage"
- moved on the sheet: C2In2, C2lp1, C3, C4, Cadc1, Cb1, Cb2, Cgnd2, D2, Dprot1, Dprot2, Dvref1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
